File: usbreset.sch (KiCad schematic (older format))
At the start: 13 parts, among them J1 USB_C_PowerSource, J2 USB_C_PowerSink, J3 USB3_A_Plug, J4 USB3_A_Receptacle, Q1 SI2393DS, SW1 EN_USBA, SW2 SW_Push, SW3 SW_Push

Commit message: Use library in schematic
Parts:
- J1, J2: footprint usbreset:10137065 -> Connector_USB-Custom:USB_C_Receptacle_Amphenol_10137065
- J4: footprint usbreset:10117835 -> Connector_USB-Custom:USB_A_Receptacle_Amphenol_10117835
- SW1: footprint usbreset:MSS3-V-T_R -> Button_Switch_SMD-Custom:SW_SPDT_MSS3-V-T_R
Changed lines of the file:
@@
 F 0 "J2" H 1507 6867 50  0000 C CNN
 F 1 "USB_C_PowerSink" H 1507 6776 50  0000 C CNN
-F 2 "usbreset:10137065" H 1550 5600 50  0001 C CNN
+F 2 "Connector_USB-Custom:USB_C_Receptacle_Amphenol_10137065" H 1550 5600 50  0001 C CNN
 F 3 "https://media.digikey.com/pdf/Data%20Sheets/Tyco%20Electonics%20AMP%20PDFs/2129691_Dwg.pdf" H 1550 5600 50  0001 C CNN
 F 4 "https://sg.element14.com/te-connectivity/2129691-1/usb-3-1-type-c-24pos-rcpt-smt/dp/2518075" H 1400 5600 50  0001 C CNN "Buy_E14"
@@
 F 0 "J1" H 1507 3367 50  0000 C CNN
 F 1 "USB_C_PowerSource" H 1507 3276 50  0000 C CNN
-F 2 "usbreset:10137065" H 1550 2100 50  0001 C CNN
+F 2 "Connector_USB-Custom:USB_C_Receptacle_Amphenol_10137065" H 1550 2100 50  0001 C CNN
 F 3 "https://media.digikey.com/pdf/Data%20Sheets/Tyco%20Electonics%20AMP%20PDFs/2129691_Dwg.pdf" H 1550 2100 50  0001 C CNN
 F 4 "https://sg.element14.com/te-connectivity/2129691-1/usb-3-1-type-c-24pos-rcpt-smt/dp/2518075" H 1400 2100 50  0001 C CNN "Buy_E14"
@@
 F 0 "SW1" H 5200 4235 50  0000 C CNN
 F 1 "EN_USBA" H 5200 4144 50  0000 C CNN
-F 2 "usbreset:MSS3-V-T_R" H 5200 4000 50  0001 C CNN
+F 2 "Button_Switch_SMD-Custom:SW_SPDT_MSS3-V-T_R" H 5200 4000 50  0001 C CNN
 F 3 "~" H 5200 4000 50  0001 C CNN
 	1    5200 4000
@@
 F 0 "J4" H 5557 6067 50  0000 C CNN
 F 1 "USB3_A_Receptacle" H 5557 5976 50  0000 C CNN
-F 2 "usbreset:10117835" H 5650 5450 50  0001 C CNN
+F 2 "Connector_USB-Custom:USB_A_Receptacle_Amphenol_10117835" H 5650 5450 50  0001 C CNN
 F 3 "~" H 5650 5450 50  0001 C CNN
 	1    5500 5350

Commit message: Initial PCB layout
Parts:
- J3: footprint (none) -> Connector_USB-Custom:USB_A_Plug_Amphenol_GSB3164x1CEU
Changed lines of the file:
@@
 F 0 "J3" H 5557 2567 50  0000 C CNN
 F 1 "USB3_A_Plug" H 5557 2476 50  0000 C CNN
-F 2 "" H 5650 1950 50  0001 C CNN
+F 2 "Connector_USB-Custom:USB_A_Plug_Amphenol_GSB3164x1CEU" H 5650 1950 50  0001 C CNN
 F 3 "~" H 5650 1950 50  0001 C CNN
 	1    5500 1850

Commit message: Route most connections
Parts:
- added R5: 0, Resistor_SMD:R_0603_1608Metric_Pad1.05x0.95mm_HandSolder, symbol Device:R
Connections:
- net GND: now also R5.2
- net SHIELD: now also R5.1
- net RX2-: now reaches J1.A10 (RX2-)
- net RX2-: now also J2.B10 (RX1-)
- net RX1+: now reaches J2.A11 (RX2+)
- net RX1+: now also J1.B11 (RX1+), J3.6 (SSRX+), J4.6 (SSRX+); no longer J1.A11 (RX2+)
- net TX1+: now reaches J1.A2 (TX1+), J3.9 (SSTX+), J4.9 (SSTX+)
- net TX1+: now also J2.B2 (TX2+); no longer J2.A2 (TX1+)
- net TX1-: now reaches J1.A3 (TX1-), J3.8 (SSTX-), J4.8 (SSTX-)
- net TX1-: now also J2.B3 (TX2-); no longer J2.A3 (TX1-)
- net CC1: now reaches J1.A5 (CC1), SW1.1 (A)
- net CC1: now also J2.B5 (CC2); no longer J2.A5 (CC1)
- net D+: now reaches J1.A6 (D+), J2.A6 (D+), J3.3 (D+), J4.3 (D+)
- net D+: now also J1.B6 (D+), J2.B6 (D+)
- net D-: now reaches J1.A7 (D-), J2.A7 (D-), J3.2 (D-), J4.2 (D-)
- net D-: now also J1.B7 (D-), J2.B7 (D-)
- net SBU1: now reaches J1.A8 (SBU1)
- net SBU1: now also J2.B8 (SBU2); no longer J2.A8 (SBU1)
- net RX1-: now reaches J1.B10 (RX1-), J3.5 (SSRX-), J4.5 (SSRX-)
- net RX1-: now also J2.A10 (RX2-); no longer J2.B10 (RX1-)
- net TX2+: now reaches J1.B2 (TX2+)
- net TX2+: now also J2.A2 (TX1+); no longer J2.B2 (TX2+)
- net TX2-: now reaches J1.B3 (TX2-)
- net TX2-: now also J2.A3 (TX1-); no longer J2.B3 (TX2-)
- net CC2: now reaches J1.B5 (CC2)
- net CC2: now also J2.A5 (CC1); no longer J2.B5 (CC2)
- net SBU2: now reaches J1.B8 (SBU2)
- net SBU2: now also J2.A8 (SBU1); no longer J2.B8 (SBU2)
- new net RX2+: J1.A11 (RX2+), J2.B11 (RX1+)

Commit message: Improve GND routing
Parts:
- J1, J2: symbol Connector:USB_C_Receptacle -> usbreset-rescue:USB_C_Receptacle-Connector
- J3, J4: symbol Connector:USB3_A -> usbreset-rescue:USB3_A-Connector
Changed lines of the file:
@@
 $EndDescr
 $Comp
-L Connector:USB_C_Receptacle J2
+L usbreset-rescue:USB_C_Receptacle-Connector J2
 U 1 1 5F157FC7
 P 1400 5600
@@
 $EndComp
 $Comp
-L Connector:USB_C_Receptacle J1
+L usbreset-rescue:USB_C_Receptacle-Connector J1
 U 1 1 5F1528AF
 P 1400 2100
@@
 VBUS_SINK
 $Comp
-L Connector:USB3_A J4
+L usbreset-rescue:USB3_A-Connector J4
 U 1 1 5FD908A9
 P 5500 5350
@@
 SHIELD
 $Comp
-L Connector:USB3_A J3
+L usbreset-rescue:USB3_A-Connector J3
 U 1 1 5FDACC9B
 P 5500 1850
